Commit message: Enabled Nav2

File: apollo_2_0/urdf/apollo_2_0.urdf (robot description, URDF)
Before this commit: robot apollo_2_0, 12 links, 11 joints
Joints:
- joint castorwheel1top: origin xyz=0.126 -0.129 0.08824 rpy=0 0 0 -> xyz=0.126 -0.129 0.0852 rpy=0 0 0
- joint castorwheel2top: origin xyz=-0.126 -0.129 0.08824 rpy=0 0 0 -> xyz=-0.126 -0.129 0.0852 rpy=0 0 0
- joint castorwheel3top: origin xyz=0.126 0.13 0.08824 rpy=0 0 0 -> xyz=0.126 0.13 0.0852 rpy=0 0 0
- joint castorwheel4top: origin xyz=-0.126 0.13 0.08824 rpy=0 0 0 -> xyz=-0.126 0.13 0.0852 rpy=0 0 0

File: apollo_2_0/urdf/apollo_2_0_gazebo.urdf.xacro (robot description, xacro)
@@ -13,5 +13,5 @@
 			</ros>
 			<!-- Plugin update rate in Hz -->
-			<update_rate>100</update_rate>
+			<update_rate>50</update_rate>
 			<num_wheel_pairs>1</num_wheel_pairs>
 			<left_joint>lw</left_joint>

File: apollo_2_0/urdf/lidar.xacro (robot description, xacro)
@@ -3,33 +3,33 @@
     <joint name="laser_joint" type="fixed">
         <parent link="base_link"/>
-        <child link="virtual_laser_frame"/>
+        <child link="laser_frame"/>
         <origin xyz="0 -0.142 0.215" rpy="0 0 0"/>
     </joint>
-    <link name="virtual_laser_frame"/>
-    <gazebo reference="virtual_laser_frame">
+    <link name="laser_frame"/>
+    <gazebo reference="laser_frame">
         <sensor name="laser" type="ray">
             <always_on>true</always_on>
             <visualize>true</visualize>
             <pose>0 0 0 0 0 0</pose>
-            <update_rate>100</update_rate>
+            <update_rate>50</update_rate>
             <ray>
-            <scan>
-                <horizontal>
-                    <samples>599.6944232238</samples> <!-- 599.6944232238 -->
-                    <resolution>1.000000</resolution>
-                    <min_angle>0.0</min_angle>
-                    <max_angle>6.28319</max_angle>
-                </horizontal>
-            </scan>
-            <range>
-                <min>0.5</min>
-                <max>10.0</max>
-                <resolution>0.015000</resolution>
-            </range>
-            <noise>
-                <type>gaussian</type>
-                <mean>0.0</mean>
-                <stddev>0.01</stddev>
-            </noise>
+                <scan>
+                    <horizontal>
+                        <samples>599.6944232238</samples> <!-- 599.6944232238 -->
+                        <resolution>1.000000</resolution>
+                        <min_angle>0.0</min_angle>
+                        <max_angle>6.28319</max_angle>
+                    </horizontal>
+                </scan>
+                <range>
+                    <min>0.5</min>
+                    <max>10.0</max>
+                    <resolution>0.015000</resolution>
+                </range>
+                <noise>
+                    <type>gaussian</type>
+                    <mean>0.0</mean>
+                    <stddev>0.01</stddev>
+                </noise>
             </ray>
             <plugin name="laser_controller" filename="libgazebo_ros_ray_sensor.so">

Commit message: FIxed Nav2 robot default front side issue

File: apollo_2_0/urdf/apollo_2_0.urdf (robot description, URDF)
Before this commit: robot apollo_2_0, 12 links, 11 joints
Links:
- added link base_footprint
Joints:
- added joint base_footprint_joint: type fixed, parent base_link, child base_footprint, origin xyz=0 0 0 rpy=0 0 -1.5708

Commit message: Corrected Base_footprint and nav2

File: apollo_2_0/urdf/apollo_2_0.urdf (robot description, URDF)
Before this commit: robot apollo_2_0, 13 links, 12 joints
Joints:
- joint base_footprint_joint: child base_footprint -> base_link; origin xyz=0 0 0 rpy=0 0 -1.5708 -> xyz=0 0 0 rpy=0 0 1.5708; parent base_link -> base_footprint

File: apollo_2_0/urdf/apollo_2_0_gazebo.urdf.xacro (robot description, xacro)
@@ -28,5 +28,5 @@
 			<odometry_frame>odom</odometry_frame>
 			<!-- Robot frame to calculate odometry from, defaults to `base_footprint` -->
-			<robot_base_frame>base_link</robot_base_frame>
+			<robot_base_frame>base_footprint</robot_base_frame>
 			<!-- Set to true to publish transforms for the odometry, defaults to true -->
 			<publish_odom>true</publish_odom>

Commit message: Correctel Castor wheels contact

File: apollo_2_0/urdf/apollo_2_0.urdf (robot description, URDF)
Before this commit: robot apollo_2_0, 13 links, 12 joints
Joints:
- joint castorwheel1top: origin xyz=0.126 -0.129 0.0852 rpy=0 0 0 -> xyz=0.126 -0.129 0.08516 rpy=0 0 0
- joint castorwheel2top: origin xyz=-0.126 -0.129 0.0852 rpy=0 0 0 -> xyz=-0.126 -0.129 0.08516 rpy=0 0 0
- joint castorwheel3top: origin xyz=0.126 0.13 0.0852 rpy=0 0 0 -> xyz=0.126 0.13 0.08516 rpy=0 0 0
- joint castorwheel4top: origin xyz=-0.126 0.13 0.0852 rpy=0 0 0 -> xyz=-0.126 0.13 0.08516 rpy=0 0 0
